File: a1200_pwr.sch (KiCad schematic (older format))
At the start: 20 parts, among them J1 PJ-102A, J2 APWR_big, J3 APWR_small, SW1 RMS1R102M7QES, U1 LMZM23600SILR, U2 RPM5.0-6.0

Commit message: Revision 2
Parts:
- U1: symbol a1200_pwr:LMZM23601SILR -> a1200_pwr-rescue:LMZM23601SILR-a1200_pwr
Changed lines of the file:
@@
 $EndDescr
 $Comp
-L a1200_pwr:LMZM23601SILR U1
+L a1200_pwr-rescue:LMZM23601SILR-a1200_pwr U1
 U 1 1 5E0DF919
 P 7750 5200
